Commit message: Fix AllegroFranka URDF left hand, Set initial arm pos

File: assets/urdf/franka_description_tmr/urdf/franka_right_digit360.urdf (robot description, URDF)
Before this commit: robot murp, 98 links, 97 joints
Links:
- link camera_front_left_link: geometry collision box size=0.026 0.124 0.029; visual mesh filename=../../realsense2_description/meshes/d455.stl scale=0.001 0.001 0.001
- link camera_front_right_link: geometry collision box size=0.026 0.124 0.029; visual mesh filename=../../realsense2_description/meshes/d455.stl scale=0.001 0.001 0.001
- link camera_rear_left_link: geometry collision box size=0.026 0.124 0.029; visual mesh filename=../../realsense2_description/meshes/d455.stl scale=0.001 0.001 0.001
- link camera_rear_right_link: geometry collision box size=0.026 0.124 0.029; visual mesh filename=../../realsense2_description/meshes/d455.stl scale=0.001 0.001 0.001
- link lidar_front: geometry collision mesh filename=../meshes_obj/nanoscan3/NANS3_collision.stl; visual mesh filename=../meshes_obj/nanoscan3/NANS3.dae
- link lidar_rear: geometry collision mesh filename=../meshes_obj/nanoscan3/NANS3_collision.stl; visual mesh filename=../meshes_obj/nanoscan3/NANS3.dae
- link link_l12.0: geometry collision box size=0.0358 0.034 0.0455; visual mesh filename=../allegro/meshes/allegro/link_12.0_left.obj
Joints:
- joint hand_left_joint: origin xyz=0 0 0.092 rpy=0 0 0.785398 -> xyz=0 0 0.092 rpy=0 0 -2.35619
- joint joint_l_12.0: axis -1 0 0 -> 1 0 0; origin xyz=-0.0182 0.019333 -0.045987 rpy=0 -1.65806278845 -1.5707963259 -> xyz=-0.0182 -0.019333 -0.045987 rpy=0 -1.65806278845 1.5707963259
- joint joint_l_13.0: axis 0 0 1 -> 0 0 -1; origin xyz=-0.027 0.005 0.0399 -> xyz=-0.027 -0.005 0.0399
- joint joint_l_4.0: axis 0 0 1 -> 0 0 -1
- joint joint_l_8.0: axis 0 0 1 -> 0 0 -1
- joint joint_l__0.0: axis 0 0 1 -> 0 0 -1
